Commit message: updated empty room asset

File: simulation/assets/scenes/empty_room/urdf/empty_room.urdf (robot description, URDF)
Before this commit: robot unnamed, 2 links, 1 joints
Links:
- removed link ground_plane
- added link wall_2; collision box size=0.10000 10.00000 1.00000; visual box size=0.10000 10.00000 1.00000
- added link wall_3; collision box size=10.00000 0.10000 1.00000; visual box size=10.00000 0.10000 1.00000
- added link wall_4; collision box size=10.00000 0.10000 1.00000; visual box size=10.00000 0.10000 1.00000
- link wall_1: geometry collision box size=0.10000 1.00000 10.00000; visual box size=0.10000 10.00000 1.00000
Joints:
- removed joint wall_1_joint
- added joint wall_1_2: type fixed, parent wall_1, child wall_2, origin xyz=0.00000 0.00000 0.00000 rpy=0.00000 0.00000 0.00000
- added joint wall_2_3: type fixed, parent wall_2, child wall_3, origin xyz=0.00000 0.00000 0.00000 rpy=0.00000 0.00000 0.00000
- added joint wall_3_4: type fixed, parent wall_3, child wall_4, origin xyz=0.00000 0.00000 0.00000 rpy=0.00000 0.00000 0.00000
