Commit message: changed walls slightly (should have no effect)

File: training_code_isaacgym/assets/scenes/empty_room_5x5/urdf/ceiled_walls_5x5x3.urdf (robot description, URDF)
Before this commit: robot unnamed, 4 links, 3 joints
Links:
- link wall_1: geometry collision box size=0.10000 3.00000 4.90000; collision box size=5.00000 5.00000 0.10000
- link wall_2: geometry collision box size=0.10000 4.90000 3.00000; visual box size=0.10000 4.90000 1.00000
- link wall_3: geometry collision box size=4.90000 0.10000 3.00000; visual box size=4.90000 0.10000 1.00000
- link wall_4: geometry collision box size=4.90000 0.10000 3.00000; visual box size=4.90000 0.10000 1.00000
