Commit message: Observations made compatible with deployment perspective.

File: training_code_isaacgym/assets/robots/go2_with_watering/urdf/go2.urdf (robot description, URDF)
Before this commit: robot go2_description, 29 links, 28 joints
Links:
- link base: mass 6.921 -> 2.

Commit message: Some rewards updated to smoother ones and additional smoothening rewards added.

File: training_code_isaacgym/assets/robots/go2_with_watering/urdf/go2.urdf (robot description, URDF)
Before this commit: robot go2_description, 29 links, 28 joints
Links:
- link base: mass 6.921 -> 2.921

Commit message: Some additional reward improvements.

File: training_code_isaacgym/assets/robots/go2_with_watering/urdf/go2.urdf (robot description, URDF)
Before this commit: robot go2_description, 29 links, 28 joints
Links:
- link base: mass 2.921 -> 2.

Commit message: Revert to working state
Revert "Reward updates and object detection probability."

This reverts commit 0699e8b62932f594888e2b9c7c952409ab4dfef8.

Revert "Merge remote-tracking branch 'origin/main'"

This reverts commit 3f46e81030306391501d8001f1d756d9382685d0, reversing
changes made to feb5bca8d13730de1fc6ec2b972fc99b263bf6e5.

File: training_code_isaacgym/assets/robots/go2_with_watering/urdf/go2.urdf (robot description, URDF)
Before this commit: robot go2_description, 29 links, 28 joints
Links:
- link base: mass 2. -> 2.921
